Commit message: update protac software repo

File: protac_description/urdf/protac_gazebo.urdf.xacro (robot description, xacro)
@@ -5,5 +5,6 @@
   <link name="world"/>
   <xacro:protac parent="world">
-    <origin xyz="0 0 0.45" rpy="0 0.785398163 0" />
+    <!-- <origin xyz="0 0 0.45" rpy="0 0.785398163 0" /> -->
+    <origin xyz="0 0 0" rpy="0 0 0" />
   </xacro:protac>
   <xacro:protac_ros2_control name="protac_ros2_control" />
