Commit message: update source files

File: protac_description/urdf/protac.urdf.xacro (robot description, xacro)
@@ -5,5 +5,5 @@
   <link name="world"/>
   <xacro:protac parent="world">
-    <origin xyz="0 0 0" rpy="0 0 0" />
+    <origin xyz="0 0 0" rpy="0 0.785398163 0" />
   </xacro:protac>
   <xacro:protac_ros2_control name="protac_ros2_control" />

File: protac_description/urdf/protac_gazebo.urdf.xacro (robot description, xacro)
@@ -5,5 +5,5 @@
   <link name="world"/>
   <xacro:protac parent="world">
-    <origin xyz="0 0 0" rpy="0 0 0" />
+    <origin xyz="0 0 0.45" rpy="0 0.785398163 0" />
   </xacro:protac>
   <xacro:protac_ros2_control name="protac_ros2_control" />

Commit message: update repo

File: protac_description/urdf/protac.urdf.xacro (robot description, xacro)
@@ -5,5 +5,6 @@
   <link name="world"/>
   <xacro:protac parent="world">
-    <origin xyz="0 0 0" rpy="0 0.785398163 0" />
+    <!-- <origin xyz="0 0 0" rpy="0 0.785398163 0" /> -->
+    <origin xyz="0 0 0.2" rpy="3.141592654 -1.570796327 0." />
   </xacro:protac>
   <xacro:protac_ros2_control name="protac_ros2_control" />

File: protac_description/urdf/protac_gazebo.urdf.xacro (robot description, xacro)
@@ -6,5 +6,5 @@
   <xacro:protac parent="world">
     <!-- <origin xyz="0 0 0.45" rpy="0 0.785398163 0" /> -->
-    <origin xyz="0 0 0" rpy="0 0 0" />
+    <origin xyz="0 0 0.2" rpy="3.141592654 -1.570796327 0." />
   </xacro:protac>
   <xacro:protac_ros2_control name="protac_ros2_control" />

File: protac_description/urdf/protac_gazebo_velocity.urdf.xacro (robot description, xacro)
@@ -5,5 +5,5 @@
   <link name="world"/>
   <xacro:protac parent="world">
-    <origin xyz="0 0 0" rpy="0 0 0" />
+    <origin xyz="0 0 0.2" rpy="3.141592654 -1.570796327 0." />
   </xacro:protac>
   <xacro:protac_ros2_control name="protac_ros2_control" />
